File: pcb/mainboard/mainboard.kicad_pcb (KiCad board)
At the start: 2 copper layers, 171.5 x 101 mm, 46 parts, among them J1 cartridge, J19 9V 1A, J2 extension_0, J3 extension_0, J4 extension_0, SW1 SW_SPST, U1 Z84C00xxP, U10 74LS244, U11 74LS244, U12 74LS244, U3 74LS283, U34 LM7805, U4 74LS00, U5 CY62256-70PC, U6 CY62256-70PC, U7 74LS138, U8 74LS244, U9 74LS244, Y1 CXO_DIP8

Commit message: .
Parts:
- removed D2: RESET, LED_THT:LED_D5.0mm
- removed J19: 9V 1A, Connector_BarrelJack:BarrelJack_Horizontal
- removed R10, R11, R12, R13: 10K, Resistor_THT:R_Axial_DIN0207_L6.3mm_D2.5mm_P7.62mm_Horizontal
- removed R5: 470R, Resistor_THT:R_Axial_DIN0207_L6.3mm_D2.5mm_P7.62mm_Horizontal
- added J18: power_jack, Connector_BarrelJack:BarrelJack_Horizontal, F.Cu at (236.2, 37.3)
- added RN1: R_Network04, Resistor_THT:R_Array_SIP5, F.Cu at (242.6, 105.4)
- added SW5: ON/OFF, power_switch:jrx, F.Cu at (210.8, 34.3)
- moved C6 188.0 mm to (69.2, 131.3), turned to 90 degrees
- moved C2 177.6 mm to (245.7, 46.3), turned to 180 degrees
- moved U6 174.6 mm to (73.7, 141.6), turned to 90 degrees
- moved D1 171.9 mm to (236.2, 46.3), turned to 180 degrees
- moved D32 164.6 mm to (226.1, 38.1), turned to 90 degrees
- moved C9 161.1 mm to (53.3, 112.3), turned to 90 degrees
- moved SW1 156.1 mm to (238.6, 52.6)
- moved U9 155.4 mm to (57.1, 114.9), turned to 90 degrees
- moved C10 145.9 mm to (90.8, 112.3), turned to 90 degrees
- moved U10 141.2 mm to (94.6, 114.9), turned to 90 degrees
- moved C13 137.5 mm to (199.4, 52.7), turned to 180 degrees
- moved C11 134.7 mm to (128.3, 112.3), turned to 90 degrees
- moved C14 134.6 mm to (189.9, 52.7)
- moved U34 131.5 mm to (190.5, 43.8)
- moved U11 131.0 mm to (132.1, 114.9), turned to 90 degrees
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Routing:
- added copper zone on B.Cu, net GND
- added copper zone on F.Cu, net GND
Other:
- board size 171.5 x 101 mm -> 218.4 x 134.6 mm
