File: pcb/mainboard/mainboard.kicad_sch (KiCad schematic)
At the start: 23 parts, among them SW1 SW_SPST, SW2 SW_DIP_x04, SW3 SW_DIP_x04, U1 Z84C00xxP, U2 74LS04, U3 74LS138, Y1 CXO_DIP8

Commit message: .
Parts:
- removed R2, R3, R8, R9: 1K, symbol Device:R
- removed R6: 470R, symbol Device:R
- removed SW2, SW3: SW_DIP_x04, symbol Switch:SW_DIP_x04
- removed U2: 74LS04, symbol 74xx:74LS04
- removed U3: 74LS138, symbol 74xx:74LS138
- added C10, C11, C12, C4, C5, C6, C7, C8, C9: 100nF, Capacitor_THT:C_Disc_D5.1mm_W3.2mm_P5.00mm, symbol Device:C
- added C13: 0.33uF, Capacitor_THT:CP_Radial_D5.0mm_P2.50mm, symbol Device:C_Polarized
- added C14: 0.1uF, Capacitor_THT:CP_Radial_D5.0mm_P2.50mm, symbol Device:C_Polarized
- added D32: 1N4001, Diode_THT:D_DO-41_SOD81_P10.16mm_Horizontal, symbol Diode:1N4001
- added J1: cartridge, edge_connector:male-edge-connector-44, symbol Connector_Generic:Conn_02x22_Top_Bottom
- added J19: 9V 1A, Connector_BarrelJack:BarrelJack_Horizontal, symbol Connector_Generic:Conn_01x02
- added J2, J3, J4: extension_0, edge_connector:male-edge-connector-44, symbol Connector_Generic:Conn_02x22_Top_Bottom
- added R10, R11, R12, R13: 10K, Resistor_THT:R_Axial_DIN0207_L6.3mm_D2.5mm_P7.62mm_Horizontal, symbol Device:R
- added U10, U11, U12, U8, U9: 74LS244, Package_DIP:DIP-20_W7.62mm, symbol 74xx:74LS244
- added U3: 74LS283, Package_DIP:DIP-16_W7.62mm, symbol 74xx:74LS283
- added U34: LM7805, Package_TO_SOT_THT:TO-220-3_Vertical, symbol Regulator_Linear:LM7805_TO220
- added U4: 74LS00, Package_DIP:DIP-14_W7.62mm, symbol 74xx:74LS00
- added U5, U6: CY62256-70PC, Package_DIP:DIP-28_W15.24mm, symbol Memory_RAM:CY62256-70PC
- added U7: 74LS138, Package_DIP:DIP-16_W7.62mm, symbol 74xx:74LS138
- C1, C2, C3: footprint (none) -> Capacitor_THT:C_Disc_D5.1mm_W3.2mm_P5.00mm
- D2: value LED -> RESET; footprint (none) -> LED_THT:LED_D5.0mm
- D3: value LED -> POWER; footprint (none) -> LED_THT:LED_D5.0mm
- D4: value LED -> HALT; footprint (none) -> LED_THT:LED_D5.0mm
- R1: value 1K -> 470R; footprint (none) -> Resistor_THT:R_Axial_DIN0207_L6.3mm_D2.5mm_P7.62mm_Horizontal
- R4, R5, R7: footprint (none) -> Resistor_THT:R_Axial_DIN0207_L6.3mm_D2.5mm_P7.62mm_Horizontal
- SW1: footprint (none) -> Button_Switch_THT:SW_PUSH_6mm
Connections:
- net +5V: now also C10.2, C11.2, C12.2, C14.1, C4.2, C5.2, C6.2, C7.2, C8.2, C9.2, J1.1 (Pin_1), J1.23 (Pin_23), J2.1 (Pin_1), J2.23 (Pin_23), J3.1 (Pin_1), J3.23 (Pin_23), J4.1 (Pin_1), J4.23 (Pin_23), U10.20 (VCC), U11.20 (VCC), U12.20 (VCC), U3.16 (VCC), U34.3 (VO), U4.14 (VCC), U5.28 (VCC), U6.28 (VCC), U7.16 (VCC), U7.6 (E3), U8.20 (VCC), U9.20 (VCC); no longer R1.1
- net GND: now also R1.1, C10.1, C11.1, C12.1, C13.2, C14.2, C4.1, C5.1, C6.1, C7.1, C8.1, C9.1, J1.22 (Pin_22), J1.44 (Pin_44), J19.2 (Pin_2), J2.22 (Pin_22), J2.44 (Pin_44), J3.22 (Pin_22), J3.44 (Pin_44), J4.22 (Pin_22), J4.44 (Pin_44), R10.1, R11.1, R12.1, R13.1, U10.10 (GND), U11.10 (GND), U12.10 (GND), U12.19 (OEb), U3.7 (C0), U3.8 (GND), U34.2 (GND), U4.7 (GND), U5.14 (GND), U6.14 (GND), U7.3 (A2), U7.4 (E1), U7.8 (GND), U8.10 (GND), U9.10 (GND)
- net ~{Z80_rfsh}: now reaches U1.28 (~{RFSH})
- net ~{Z80_rfsh}: now also U12.13 (I1b)
- net at C2.1, D1.2 (A), R4.2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: now also U4.1, U4.2
- net at R5.1: now also U4.10, U4.3, U4.9
- net at D3.1 (K): now also R1.2
- net ~{Z80_busack}: now reaches U1.23 (~{BUSACK})
- net ~{Z80_busack}: now also U12.15 (I2b), U4.12, U4.13
- net ~{Z80_nmi}: now reaches U1.17 (~{NMI})
- net ~{Z80_nmi}: now also J2.41 (Pin_41), J3.41 (Pin_41), J4.41 (Pin_41); no longer R1.2
- net ~{Z80_wait}: now reaches U1.24 (~{WAIT})
- net ~{Z80_wait}: now also J2.43 (Pin_43), J3.43 (Pin_43), J4.43 (Pin_43)
- net ~{Z80_busreq}: now reaches U1.25 (~{BUSREQ})
- net ~{Z80_busreq}: now also J2.38 (Pin_38), J3.38 (Pin_38), J4.38 (Pin_38)
- net A0 renamed Z80_addr_{0}
- net Z80_addr_{0}: now also U8.2 (I0a)
- net A1 renamed Z80_addr_{1}
- net Z80_addr_{1}: now also U8.4 (I1a)
- net A10 renamed Z80_addr_{10}
- net Z80_addr_{10}: now also U10.6 (I2a)
- net A11 renamed Z80_addr_{11}
- net Z80_addr_{11}: now also U10.8 (I3a)
- net A12 renamed Z80_addr_{12}
- net Z80_addr_{12}: now also U10.11 (I0b)
- net A13 renamed Z80_addr_{13}
- net Z80_addr_{13}: now also U10.13 (I1b)
- net A14 renamed Z80_addr_{14}
- net Z80_addr_{14}: now also U10.15 (I2b)
- net A15 renamed Z80_addr_{15}
- net Z80_addr_{15}: now also U10.17 (I3b)
- net A2 renamed Z80_addr_{2}
- net Z80_addr_{2}: now also U8.6 (I2a)
- net A3 renamed Z80_addr_{3}
- net Z80_addr_{3}: now also U8.8 (I3a)
- net A4 renamed Z80_addr_{4}
- net Z80_addr_{4}: now also U8.11 (I0b)
- net A5 renamed Z80_addr_{5}
- net Z80_addr_{5}: now also U8.13 (I1b)
- net A6 renamed Z80_addr_{6}
- net Z80_addr_{6}: now also U8.15 (I2b)
- net A7 renamed Z80_addr_{7}
- net Z80_addr_{7}: now also U8.17 (I3b)
- net A8 renamed Z80_addr_{8}
- net Z80_addr_{8}: now also U10.2 (I0a)
- net A9 renamed Z80_addr_{9}
- net Z80_addr_{9}: now also U10.4 (I1a)
- net D0 renamed Z80_data_{0}
- net Z80_data_{0}: now also U11.18 (O0a), U9.2 (I0a)
- net D1 renamed Z80_data_{1}
- net Z80_data_{1}: now also U11.16 (O1a), U9.4 (I1a)
- net D2 renamed Z80_data_{2}
- net Z80_data_{2}: now also U11.14 (O2a), U9.6 (I2a)
- net D3 renamed Z80_data_{3}
- net Z80_data_{3}: now also U11.12 (O3a), U9.8 (I3a)
- net D4 renamed Z80_data_{4}
- net Z80_data_{4}: now also U11.9 (O0b), U9.11 (I0b)
- net D5 renamed Z80_data_{5}
- net Z80_data_{5}: now also U11.7 (O1b), U9.13 (I1b)
- net D6 renamed Z80_data_{6}
- net Z80_data_{6}: now also U11.5 (O2b), U9.15 (I2b)
- net D7 renamed Z80_data_{7}
- net Z80_data_{7}: now also U11.3 (O3b), U9.17 (I3b)
- net clock renamed Z80_clock
- net ~{halt} renamed ~{Z80_halt}
- net ~{Z80_halt}: now also U12.17 (I3b); no longer R7.1
- net ~{int} renamed ~{Z80_int}
- net ~{Z80_int}: now also J2.40 (Pin_40), J3.40 (Pin_40), J4.40 (Pin_40)
- net ~{iorq} renamed ~{Z80_iorq}
- net ~{Z80_iorq}: now also U12.4 (I1a)
- net ~{m1} renamed ~{Z80_m1}
- net ~{Z80_m1}: now also U12.11 (I0b)
- net ~{mreq} renamed ~{Z80_mreq}
- net ~{Z80_mreq}: now also U12.2 (I0a)
- net ~{rd} renamed ~{Z80_rd}
- net ~{Z80_rd}: now also U12.6 (I2a)
- net ~{reset} renamed ~{Z80_reset}
- net ~{Z80_reset}: now also U4.8
- net ~{wr} renamed ~{Z80_wr}
- net ~{Z80_wr}: now also U12.8 (I3a)
- new net: C13.1, D32.1 (K), U34.1 (VI)
- new net: U4.4, U7.13 (O2)
- new net: U4.5, U7.12 (O3)
- new net: D32.2 (A), J19.1 (Pin_1)
- new net addr_sel_{0}: J1.40 (Pin_40), R10.2, U3.5 (A1)
- new net addr_sel_{1}: J1.41 (Pin_41), R11.2, U3.3 (A2)
- new net addr_sel_{2}: J1.42 (Pin_42), R12.2, U3.14 (A3)
- new net addr_sel_{3}: J1.43 (Pin_43), R13.2, U3.12 (A4)
- new net bus_addr_{0}: J1.6 (Pin_6), J2.6 (Pin_6), J3.6 (Pin_6), J4.6 (Pin_6), U5.10 (A0), U6.10 (A0), U8.18 (O0a)
- new net bus_addr_{10}: J1.16 (Pin_16), J2.16 (Pin_16), J3.16 (Pin_16), J4.16 (Pin_16), U10.14 (O2a), U5.21 (A10), U6.21 (A10)
- new net bus_addr_{11}: J1.17 (Pin_17), J2.17 (Pin_17), J3.17 (Pin_17), J4.17 (Pin_17), U10.12 (O3a), U5.23 (A11), U6.23 (A11)
- new net bus_addr_{12}: J1.18 (Pin_18), J2.18 (Pin_18), J3.18 (Pin_18), J4.18 (Pin_18), U10.9 (O0b), U3.6 (B1), U5.2 (A12), U6.2 (A12)
- new net bus_addr_{13}: J1.19 (Pin_19), J2.19 (Pin_19), J3.19 (Pin_19), J4.19 (Pin_19), U10.7 (O1b), U3.2 (B2), U5.26 (A13), U6.26 (A13)
- new net bus_addr_{14}: J1.20 (Pin_20), J2.20 (Pin_20), J3.20 (Pin_20), J4.20 (Pin_20), U10.5 (O2b), U3.15 (B3), U5.1 (A14), U6.1 (A14)
- new net bus_addr_{15}: J1.21 (Pin_21), J2.21 (Pin_21), J3.21 (Pin_21), J4.21 (Pin_21), U10.3 (O3b), U3.11 (B4), U7.1 (A0)
- new net bus_addr_{1}: J1.7 (Pin_7), J2.7 (Pin_7), J3.7 (Pin_7), J4.7 (Pin_7), U5.9 (A1), U6.9 (A1), U8.16 (O1a)
- new net bus_addr_{2}: J1.8 (Pin_8), J2.8 (Pin_8), J3.8 (Pin_8), J4.8 (Pin_8), U5.8 (A2), U6.8 (A2), U8.14 (O2a)
- new net bus_addr_{3}: J1.9 (Pin_9), J2.9 (Pin_9), J3.9 (Pin_9), J4.9 (Pin_9), U5.7 (A3), U6.7 (A3), U8.12 (O3a)
- new net bus_addr_{4}: J1.10 (Pin_10), J2.10 (Pin_10), J3.10 (Pin_10), J4.10 (Pin_10), U5.6 (A4), U6.6 (A4), U8.9 (O0b)
- new net bus_addr_{5}: J1.11 (Pin_11), J2.11 (Pin_11), J3.11 (Pin_11), J4.11 (Pin_11), U5.5 (A5), U6.5 (A5), U8.7 (O1b)
- new net bus_addr_{6}: J1.12 (Pin_12), J2.12 (Pin_12), J3.12 (Pin_12), J4.12 (Pin_12), U5.4 (A6), U6.4 (A6), U8.5 (O2b)
- new net bus_addr_{7}: J1.13 (Pin_13), J2.13 (Pin_13), J3.13 (Pin_13), J4.13 (Pin_13), U5.3 (A7), U6.3 (A7), U8.3 (O3b)
- new net bus_addr_{8}: J1.14 (Pin_14), J2.14 (Pin_14), J3.14 (Pin_14), J4.14 (Pin_14), U10.18 (O0a), U5.25 (A8), U6.25 (A8)
- new net bus_addr_{9}: J1.15 (Pin_15), J2.15 (Pin_15), J3.15 (Pin_15), J4.15 (Pin_15), U10.16 (O1a), U5.24 (A9), U6.24 (A9)
- new net bus_busack: U10.1 (OEa), U10.19 (OEb), U11.1 (OEa), U11.19 (OEb), U12.1 (OEa), U4.11, U8.1 (OEa), U8.19 (OEb), U9.1 (OEa), U9.19 (OEb)
- new net bus_clock: J2.33 (Pin_33), J3.33 (Pin_33), J4.33 (Pin_33)
- new net bus_data_{0}: J1.24 (Pin_24), J2.24 (Pin_24), J3.24 (Pin_24), J4.24 (Pin_24), U11.2 (I0a), U5.11 (Q0), U6.11 (Q0), U9.18 (O0a)
- new net bus_data_{1}: J1.25 (Pin_25), J2.25 (Pin_25), J3.25 (Pin_25), J4.25 (Pin_25), U11.4 (I1a), U5.12 (Q1), U6.12 (Q1), U9.16 (O1a)
- new net bus_data_{2}: J1.26 (Pin_26), J2.26 (Pin_26), J3.26 (Pin_26), J4.26 (Pin_26), U11.6 (I2a), U5.13 (Q2), U6.13 (Q2), U9.14 (O2a)
- new net bus_data_{3}: J1.27 (Pin_27), J2.27 (Pin_27), J3.27 (Pin_27), J4.27 (Pin_27), U11.8 (I3a), U5.15 (Q3), U6.15 (Q3), U9.12 (O3a)
- new net bus_data_{4}: J1.28 (Pin_28), J2.28 (Pin_28), J3.28 (Pin_28), J4.28 (Pin_28), U11.11 (I0b), U5.16 (Q4), U6.16 (Q4), U9.9 (O0b)
- new net bus_data_{5}: J1.29 (Pin_29), J2.29 (Pin_29), J3.29 (Pin_29), J4.29 (Pin_29), U11.13 (I1b), U5.17 (Q5), U6.17 (Q5), U9.7 (O1b)
- new net bus_data_{6}: J1.30 (Pin_30), J2.30 (Pin_30), J3.30 (Pin_30), J4.30 (Pin_30), U11.15 (I2b), U5.18 (Q6), U6.18 (Q6), U9.5 (O2b)
- new net bus_data_{7}: J1.31 (Pin_31), J2.31 (Pin_31), J3.31 (Pin_31), J4.31 (Pin_31), U11.17 (I3b), U5.19 (Q7), U6.19 (Q7), U9.3 (O3b)
- new net rom_address: U3.9 (C4), U7.2 (A1)
- new net rom_select: J1.3 (Pin_3), U4.6
- new net ~{bus_busack}: J2.39 (Pin_39), J3.39 (Pin_39), J4.39 (Pin_39), U12.5 (O2b)
- new net ~{bus_halt}: J2.42 (Pin_42), J3.42 (Pin_42), J4.42 (Pin_42), R7.1, U12.3 (O3b)
- new net ~{bus_iorq}: J2.36 (Pin_36), J3.36 (Pin_36), J4.36 (Pin_36), U12.16 (O1a)
- new net ~{bus_m1}: J2.34 (Pin_34), J3.34 (Pin_34), J4.34 (Pin_34), U12.9 (O0b)
- new net ~{bus_mreq}: J2.35 (Pin_35), J3.35 (Pin_35), J4.35 (Pin_35), U12.18 (O0a), U7.5 (E2)
- new net ~{bus_rd}: J1.5 (Pin_5), J2.5 (Pin_5), J3.5 (Pin_5), J4.5 (Pin_5), U12.14 (O2a), U5.22 (~{OE}), U6.22 (~{OE})
- new net ~{bus_rfsh}: J2.37 (Pin_37), J3.37 (Pin_37), J4.37 (Pin_37), U12.7 (O1b)
- new net ~{bus_wr}: J1.4 (Pin_4), J2.4 (Pin_4), J3.4 (Pin_4), J4.4 (Pin_4), U12.12 (O3a), U5.27 (~{WE}), U6.27 (~{WE})
- new net ~{ram_0_select}: U5.20 (~{CS}), U7.15 (O0)
- new net ~{ram_1_select}: U6.20 (~{CS}), U7.14 (O1)
- no-connect marks 1 -> 27
Other:
- moved on the sheet: C1, D4, R7, U1

Commit message: .
Parts:
- removed D2: RESET, LED_THT:LED_D5.0mm, symbol Device:LED
- removed J19: 9V 1A, Connector_BarrelJack:BarrelJack_Horizontal, symbol Connector_Generic:Conn_01x02
- removed R10, R11, R12, R13: 10K, Resistor_THT:R_Axial_DIN0207_L6.3mm_D2.5mm_P7.62mm_Horizontal, symbol Device:R
- removed R5: 470R, Resistor_THT:R_Axial_DIN0207_L6.3mm_D2.5mm_P7.62mm_Horizontal, symbol Device:R
- added J18: power_jack, Connector_BarrelJack:BarrelJack_Horizontal, symbol Connector:Barrel_Jack_Switch
- added J5: extension_3, edge_connector:male-edge-connector-44, symbol Connector_Generic:Conn_02x22_Top_Bottom
- added RN1: R_Network04, Resistor_THT:R_Array_SIP5, symbol Device:R_Network04
- added SW5: ON/OFF, power_switch:jrx, symbol Switch:SW_SPST
- J3: value extension_0 -> extension_1
- J4: value extension_0 -> extension_2
Connections:
- net +5V: now also J5.1 (Pin_1), J5.23 (Pin_23)
- net GND: now also J18.1, J5.22 (Pin_22), J5.44 (Pin_44), RN1.1 (common)
- net addr_sel_{0}: now also RN1.5 (R4)
- net addr_sel_{1}: now also RN1.4 (R3)
- net addr_sel_{2}: now also RN1.3 (R2)
- net addr_sel_{3}: now also RN1.2 (R1)
- net bus_addr_{0}: now also J5.6 (Pin_6)
- net bus_addr_{10}: now also J5.16 (Pin_16)
- net bus_addr_{11}: now also J5.17 (Pin_17)
- net bus_addr_{12}: now also J5.18 (Pin_18)
- net bus_addr_{13}: now also J5.19 (Pin_19)
- net bus_addr_{14}: now also J5.20 (Pin_20)
- net bus_addr_{15}: now also J5.21 (Pin_21)
- net bus_addr_{1}: now also J5.7 (Pin_7)
- net bus_addr_{2}: now also J5.8 (Pin_8)
- net bus_addr_{3}: now also J5.9 (Pin_9)
- net bus_addr_{4}: now also J5.10 (Pin_10)
- net bus_addr_{5}: now also J5.11 (Pin_11)
- net bus_addr_{6}: now also J5.12 (Pin_12)
- net bus_addr_{7}: now also J5.13 (Pin_13)
- net bus_addr_{8}: now also J5.14 (Pin_14)
- net bus_addr_{9}: now also J5.15 (Pin_15)
- net bus_busack: no longer U11.1 (OEa), U11.19 (OEb), U9.1 (OEa), U9.19 (OEb)
- net bus_clock: now also J5.33 (Pin_33)
- net bus_data_{0}: now also J5.24 (Pin_24)
- net bus_data_{1}: now also J5.25 (Pin_25)
- net bus_data_{2}: now also J5.26 (Pin_26)
- net bus_data_{3}: now also J5.27 (Pin_27)
- net bus_data_{4}: now also J5.28 (Pin_28)
- net bus_data_{5}: now also J5.29 (Pin_29)
- net bus_data_{6}: now also J5.30 (Pin_30)
- net bus_data_{7}: now also J5.31 (Pin_31)
- net ~{Z80_busreq}: now also J5.38 (Pin_38)
- net ~{Z80_int}: now also J5.40 (Pin_40)
- net ~{Z80_nmi}: now also J5.41 (Pin_41)
- net ~{Z80_rd}: now also U11.1 (OEa), U11.19 (OEb)
- net ~{Z80_wait}: now also J5.43 (Pin_43)
- net ~{Z80_wr}: now also U9.1 (OEa), U9.19 (OEb)
- net ~{bus_busack}: now also J5.39 (Pin_39)
- net ~{bus_halt}: now also J5.42 (Pin_42)
- net ~{bus_iorq}: now also J5.36 (Pin_36)
- net ~{bus_m1}: now also J5.34 (Pin_34)
- net ~{bus_mreq}: now also J5.35 (Pin_35)
- net ~{bus_rd}: now also J5.5 (Pin_5)
- net ~{bus_rfsh}: now also J5.37 (Pin_37)
- net ~{bus_wr}: now also J5.4 (Pin_4)
- net at D32.2 (A): now also SW5.1 (A)
- new net: J18.2, SW5.2 (B)
- no-connect marks 27 -> 31
Other:
- moved on the sheet: C10, C11, C12, C13, C14, C5, C6, C8, C9, D32, U10, U11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
